Commit message: Add diff_drive controller and finish urdf

File: differential_bot/description/lidar.xacro (robot description, xacro)
@@ -22,35 +22,3 @@
         </xacro:inertial_cylinder>
     </link>
-    <!-- CONTROL -->
-    <gazebo reference="laser_frame">
-        <material>Gazebo/White</material>
-        <sensor type="ray" name="head_hokuyo_sensor">
-            <pose> 0 0 0 0 0 0 </pose>
-            <visualize>true</visualize>
-            <update_rate>5.5</update_rate>
-            <ray>
-                <scan>
-                    <horizontal>
-                        <samples>360</samples>
-                        <resolution>1</resolution>
-                        <min_angle>-${pi}</min_angle>
-                        <max_angle>${pi}</max_angle>
-                    </horizontal>
-                </scan>
-                <range>
-                    <min>0.3</min>
-                    <max>12</max> <!-- 6 realistically -->
-                </range>
-                <noise>
-                    <type>gaussian</type>
-                    <mean>0.0</mean>
-                    <stddev>0.01</stddev>
-                </noise>
-            </ray>
-            <plugin name="gazebo_ros_head_hokuyo_controller" filename="libgazebo_ros_laser.so">
-                <topicName>/scan</topicName>
-                <frameName>laser_frame</frameName>
-            </plugin>
-        </sensor>
-    </gazebo>
 </robot>

File: differential_bot/description/robot_core.xacro (robot description, xacro)
@@ -65,4 +65,14 @@
         </xacro:inertial_cylinder>
     </link>
+    <transmission name="left_wheel_transmission">
+        <type>transmission_interface/SimpleTransmission</type>
+        <joint name="left_wheel_joint">
+            <hardwareInterface>hardware_interface/VelocityJointInterface</hardwareInterface>
+        </joint>
+        <actuator name="left_wheel_actuator">
+            <mechanicalReduction>7</mechanicalReduction>
+            <hardwareInterface>VelocityJointInterface</hardwareInterface>
+        </actuator>
+    </transmission>
     <gazebo reference="left_wheel">
         <material>Gazebo/Red</material>
@@ -93,4 +103,14 @@
         </xacro:inertial_cylinder>
     </link>
+    <transmission name="right_wheel_transmission">
+        <type>transmission_interface/SimpleTransmission</type>
+        <joint name="right_wheel_joint">
+            <hardwareInterface>hardware_interface/VelocityJointInterface</hardwareInterface>
+        </joint>
+        <actuator name="right_wheel_actuator">
+            <mechanicalReduction>7</mechanicalReduction>
+            <hardwareInterface>VelocityJointInterface</hardwareInterface>
+        </actuator>
+    </transmission>
     <gazebo reference="right_wheel">
         <material>Gazebo/Red</material>
@@ -125,6 +145,7 @@
         <mu2 value="0.001"/>
     </gazebo>
-    <!-- <gazebo>
-        <plugin name="gazebo_ros_control" filename="libgazebo_ros_contol.so" />
-    </gazebo> -->
+    <gazebo>
+        <plugin name="gazebo_ros_control" filename="libgazebo_ros_control.so" >
+        </plugin>
+    </gazebo>
 </robot>

File: differential_bot/description/robot_gazebo.urdf.xacro (robot description, xacro)
@@ -2,5 +2,6 @@
 <robot xmlns:xacro="http://www.ros.org/wiki/xacro" name="robot">
     <xacro:include filename="robot_core.xacro"/>
-    <xacro:include filename="diff_drive_controller.xacro"/>
+    <!-- <xacro:include filename="diff_drive_controller.xacro"/> -->
     <xacro:include filename="lidar.xacro"/>
+    <xacro:include filename="gazebo.xacro"/>
 </robot>
